Commit message: cleanup

File: zuros_hardware_config/zuros/urdf/zuros.urdf (robot description, URDF)
Before this commit: robot zuros, 10 links, 9 joints
Links:
- removed link base_battery_link
- removed link left_back_wheel
- removed link left_back_wheel_swivel_left
- removed link left_back_wheel_swivel_right
- removed link left_front_wheel
- removed link right_back_wheel
- removed link right_back_wheel_swivel_left
- removed link right_back_wheel_swivel_right
- removed link right_front_wheel
- added link base_laser; visual box size=0.035 0.18 0.024
- link base_link: geometry visual box size=0.565 0.456 0.083
Joints:
- removed joint base_battery_joint
- removed joint left_back_wheel_joint
- removed joint left_back_wheel_left_swivel_joint
- removed joint left_back_wheel_right_swivel_joint
- removed joint left_front_wheel_joint
- removed joint right_back_wheel_joint
- removed joint right_back_wheel_left_swivel_joint
- removed joint right_back_wheel_right_swivel_joint
- removed joint right_front_wheel_joint
- added joint base_to_laser: type fixed, parent base_link, child base_laser

Commit message: further testing

File: zuros_hardware_config/zuros/urdf/zuros.urdf (robot description, URDF)
Before this commit: robot zuros, 2 links, 1 joints
Joints:
- joint base_to_laser: origin (none) -> xyz=0.2745 0 -0.0775
